Commit message: fix: optimization fixes on rendered bugs within robot arm, now simulates with primitive hitboxes but with visuals .stl files

File: lbr_description/models/ft_sensor/real_ft_sensor_macro.xacro (robot description, xacro)
@@ -40,5 +40,7 @@
 		<origin xyz="0 0 0" rpy="0 0 0"/>
 		<geometry>
-			<mesh filename="package://lbr_description/models/brida/meshes/collision/brida_cam.stl"/>
+		<!--- ahora usa un cilindro primitivo para optimizar los golpes y el calculo de colisiones -->
+		<!-- <mesh filename="package://lbr_description/models/brida/meshes/collision/brida_cam.stl"/> -->
+			<cylinder radius="0.031" length="0.01"/>
 		</geometry>
 	</collision>
@@ -76,5 +78,7 @@
 		<origin xyz="0 0 0" rpy="0 0 0"/>
 		<geometry>
-			<mesh filename="package://lbr_description/models/ft_sensor/meshes/collision/FT45.stl"/>
+		<cylinder radius="0.0225" length="0.021"/>
+		<!--- la parte de arriba ya han llegado a usar formas primitivas para ahorrar CPU -->
+		<!--- 	<mesh filename="package://lbr_description/models/ft_sensor/meshes/collision/FT45.stl"/> -->
 		</geometry>
 	</collision>
@@ -112,5 +116,6 @@
 		<origin xyz="0 0 0" rpy="0 0 0"/>
 		<geometry>
-			<mesh filename="package://lbr_description/models/brida/meshes/collision/brida_ft.stl"/>
+		    <cylinder radius="0.022" length="0.01"/>
+			<!-- <mesh filename="package://lbr_description/models/brida/meshes/collision/brida_ft.stl"/> -->
 		</geometry>
 	</collision>

File: lbr_description/models/tool/tool.xacro (robot description, xacro)
@@ -98,5 +98,8 @@
           <origin xyz="0 0 0" rpy="0 0 0" />
           <geometry>
-            <mesh filename="package://lbr_description/models/tool/meshes/collision/tool_base.stl"/>
+          <!--- forma primitiva para optimizar CPU, calculos propios -->
+          <!-- TODO: revisar las dimensiones del cilindro para que se ajusten a la realidad -->
+            <cylinder radius="0.075" length="0.10" />
+            <!-- <mesh filename="package://lbr_description/models/tool/meshes/collision/tool_base.stl"/> -->
           </geometry>
         </collision>
@@ -130,5 +133,8 @@
           <origin xyz="0 0 0" rpy="0 0 0" />
           <geometry>
-            <mesh filename="package://lbr_description/models/tool/meshes/collision/tool_sponge_red.stl"/>
+          <!--- forma primitiva para optimizar CPU, calculos propios -->
+          <!-- TODO: revisar las dimensiones del cilindro para que se ajusten a la realidad -->
+            <cylinder radius="0.075" length="0.0524" />
+            <!-- <mesh filename="package://lbr_description/models/tool/meshes/collision/tool_sponge_red.stl"/> -->
           </geometry>
         </collision>

File: lbr_description/urdf/iiwa7/iiwa7.xacro (robot description, xacro)
@@ -66,9 +66,9 @@
             </geometry>
         </visual>
+        <!-- caja simplificada para tratar de optimizar el codigo -->
         <collision>
-            <origin xyz="0 0 0" rpy="0 0 0" />
+            <origin xyz="0.0 0.0 -0.1685" rpy="0 0 0" />
             <geometry>
-                <mesh filename="package://lbr_description/meshes/iiwa7/carrito_azul/Cuerpo_carro_1.stl"
-                      scale="0.001 0.001 0.001" />
+                <box size="1.055 0.705 0.983" />
             </geometry>
         </collision>
@@ -102,5 +102,6 @@
     <xacro:ft_gazebo_plugin
         ft_joint_name="brida_cam_tip_ft45_base_joint"
-        topic_name="ft_sensor/wrench" />
+        topic_name="ft_sensor/wrench"
+        update_rate="200"/> <!-- bajado la frecuencia de actualizacion para optimizar, sin cambios -->
     <xacro:brida_ft
         parent="ft45_tip"
@@ -116,7 +117,9 @@
         name="tool"
         parent="tool_body_tip">
-        <origin xyz="0 0 0" rpy="0 0 0" />
+        <origin xyz="0 0 0" rpy="0 0 ${pi}" />
     </xacro:repair_sponge_red>
     <!-- TCP alternativo fijo desde link_7 para IK -->
+    <!-- no uso el dummy para que no haya una duplicidad de los puntos TCP, sin cambios, no funciona la optimizacion igualmente -->
+    <!--
     <link name="tool_tip_dummy" />
     <joint name="$(arg robot_name)_link_7-tool_tip_dummy" type="fixed">
@@ -125,3 +128,4 @@
         <origin xyz="0 0 0" rpy="0 0 ${pi}" />
     </joint>
+    -->
 </robot>
