Commit message: feat: new gazebo implementations for code related optimizations and topics

File: lbr_description/urdf/iiwa7/iiwa7.urdf.xacro (robot description, xacro)
@@ -1,9 +1,14 @@
-<?xml version="1.0"?>
+<?xml version="1.0" ?>
 <robot xmlns:xacro="http://www.ros.org/wiki/xacro">
     <!-- robot as extracted via https://github.com/syuntoku14/fusion2urdf -->
-    <xacro:macro name="iiwa7"
-        params="robot_name:=^|lbr joint_limits_path:=^|'$(find lbr_description)/urdf/iiwa7/joint_limits.yaml'">
+    <xacro:macro
+        name="iiwa7"
+        params="robot_name:=^|lbr joint_limits_path:=^|'$(find lbr_description)/urdf/iiwa7/joint_limits.yaml'"
+    >
         <!-- load joint limits via yaml -->
-        <xacro:property name="joint_limits" value="${xacro.load_yaml(joint_limits_path)}" />
+        <xacro:property
+            name="joint_limits"
+            value="${xacro.load_yaml(joint_limits_path)}"
+        />
         <!-- constants -->
         <xacro:property name="PI" value="3.1415926535897931" />
@@ -15,11 +20,19 @@
                 <origin rpy="0 0 0" xyz="-0.012857 0.0 0.069964" />
                 <mass value="4.855658" />
-                <inertia ixx="0.017839" ixy="0.0" ixz="0.000781" iyy="0.022294" iyz="0.0"
-                    izz="0.021334" />
+                <inertia
+                    ixx="0.017839"
+                    ixy="0.0"
+                    ixz="0.000781"
+                    iyy="0.022294"
+                    iyz="0.0"
+                    izz="0.021334"
+                />
             </inertial>
             <visual>
                 <origin rpy="0 0 0" xyz="0 0 0" />
                 <geometry>
-                    <mesh filename="package://lbr_description/meshes/iiwa7/visual/link_0.dae" />
+                    <mesh
+                        filename="package://lbr_description/meshes/iiwa7/visual/link_0.dae"
+                    />
                 </geometry>
             </visual>
@@ -27,5 +40,7 @@
                 <origin rpy="0 0 0" xyz="0 0 0" />
                 <geometry>
-                    <mesh filename="package://lbr_description/meshes/iiwa7/collision/link_0.stl" />
+                    <mesh
+                        filename="package://lbr_description/meshes/iiwa7/collision/link_0.stl"
+                    />
                 </geometry>
             </collision>
@@ -40,10 +55,12 @@
                 lower="${joint_limits['A1']['lower'] * PI / 180}"
                 upper="${joint_limits['A1']['upper'] * PI / 180}"
-                velocity="${joint_limits['A1']['velocity'] * PI / 180}" />
+                velocity="${joint_limits['A1']['velocity'] * PI / 180}"
+            />
             <safety_controller
                 soft_lower_limit="${joint_limits['A1']['lower'] * PI / 180}"
                 soft_upper_limit="${joint_limits['A1']['upper'] * PI / 180}"
                 k_position="${joint_limits['A1']['velocity'] / joint_limits['A1']['safety_position_margin']}"
-                k_velocity="${joint_limits['A1']['k_velocity']}" />
+                k_velocity="${joint_limits['A1']['k_velocity']}"
+            />
             <dynamics damping="${joint_damping}" friction="${joint_friction}" />
         </joint>
@@ -52,11 +69,19 @@
                 <origin rpy="0 0 0" xyz="0.0 -0.034819 0.123299" />
                 <mass value="3.394011" />
-                <inertia ixx="0.021383" ixy="0.0" ixz="0.0" iyy="0.020403" iyz="0.003797"
-                    izz="0.007563" />
+                <inertia
+                    ixx="0.021383"
+                    ixy="0.0"
+                    ixz="0.0"
+                    iyy="0.020403"
+                    iyz="0.003797"
+                    izz="0.007563"
+                />
             </inertial>
             <visual>
                 <origin rpy="0 0 0" xyz="0.0 0.0 -0.1475" />
                 <geometry>
-                    <mesh filename="package://lbr_description/meshes/iiwa7/visual/link_1.dae" />
+                    <mesh
+                        filename="package://lbr_description/meshes/iiwa7/visual/link_1.dae"
+                    />
                 </geometry>
             </visual>
@@ -64,5 +89,7 @@
                 <origin rpy="0 0 0" xyz="0.0 0.0 -0.1475" />
                 <geometry>
-                    <mesh filename="package://lbr_description/meshes/iiwa7/collision/link_1.stl" />
+                    <mesh
+                        filename="package://lbr_description/meshes/iiwa7/collision/link_1.stl"
+                    />
                 </geometry>
             </collision>
@@ -77,10 +104,12 @@
                 lower="${joint_limits['A2']['lower'] * PI / 180}"
                 upper="${joint_limits['A2']['upper'] * PI / 180}"
-                velocity="${joint_limits['A2']['velocity'] * PI / 180}" />
+                velocity="${joint_limits['A2']['velocity'] * PI / 180}"
+            />
             <safety_controller
                 soft_lower_limit="${joint_limits['A2']['lower'] * PI / 180}"
                 soft_upper_limit="${joint_limits['A2']['upper'] * PI / 180}"
                 k_position="${joint_limits['A2']['velocity'] / joint_limits['A2']['safety_position_margin']}"
-                k_velocity="${joint_limits['A2']['k_velocity']}" />
+                k_velocity="${joint_limits['A2']['k_velocity']}"
+            />
             <dynamics damping="${joint_damping}" friction="${joint_friction}" />
         </joint>
@@ -89,11 +118,19 @@
                 <origin rpy="0 0 0" xyz="0.0 0.039793 0.086944" />
                 <mass value="4.031991" />
-                <inertia ixx="0.031697" ixy="0.0" ixz="0.0" iyy="0.03008" iyz="0.005889"
-                    izz="0.009666" />
+                <inertia
+                    ixx="0.031697"
+                    ixy="0.0"
+                    ixz="0.0"
+                    iyy="0.03008"
+                    iyz="0.005889"
+                    izz="0.009666"
+                />
             </inertial>
             <visual>
                 <origin rpy="0 0 0" xyz="0.0 0.0105 -0.34" />
                 <geometry>
-                    <mesh filename="package://lbr_description/meshes/iiwa7/visual/link_2.dae" />
+                    <mesh
+                        filename="package://lbr_description/meshes/iiwa7/visual/link_2.dae"
+                    />
                 </geometry>
             </visual>
@@ -101,5 +138,7 @@
                 <origin rpy="0 0 0" xyz="0.0 0.0105 -0.34" />
                 <geometry>
-                    <mesh filename="package://lbr_description/meshes/iiwa7/collision/link_2.stl" />
+                    <mesh
+                        filename="package://lbr_description/meshes/iiwa7/collision/link_2.stl"
+                    />
                 </geometry>
             </collision>
@@ -114,10 +153,12 @@
                 lower="${joint_limits['A3']['lower'] * PI / 180}"
                 upper="${joint_limits['A3']['upper'] * PI / 180}"
-                velocity="${joint_limits['A3']['velocity'] * PI / 180}" />
+                velocity="${joint_limits['A3']['velocity'] * PI / 180}"
+            />
             <safety_controller
                 soft_lower_limit="${joint_limits['A3']['lower'] * PI / 180}"
                 soft_upper_limit="${joint_limits['A3']['upper'] * PI / 180}"
                 k_position="${joint_limits['A3']['velocity'] / joint_limits['A3']['safety_position_margin']}"
-                k_velocity="${joint_limits['A3']['k_velocity']}" />
+                k_velocity="${joint_limits['A3']['k_velocity']}"
+            />
             <dynamics damping="${joint_damping}" friction="${joint_friction}" />
         </joint>
@@ -126,11 +167,19 @@
                 <origin rpy="0 0 0" xyz="0.0 0.034819 0.123299" />
                 <mass value="3.394011" />
-                <inertia ixx="0.021383" ixy="0.0" ixz="0.0" iyy="0.020403" iyz="-0.003797"
-                    izz="0.007563" />
+                <inertia
+                    ixx="0.021383"
+                    ixy="0.0"
+                    ixz="0.0"
+                    iyy="0.020403"
+                    iyz="-0.003797"
+                    izz="0.007563"
+                />
             </inertial>
             <visual>
                 <origin rpy="0 0 0" xyz="0.0 0.0 -0.5475" />
                 <geometry>
-                    <mesh filename="package://lbr_description/meshes/iiwa7/visual/link_3.dae" />
+                    <mesh
+                        filename="package://lbr_description/meshes/iiwa7/visual/link_3.dae"
+                    />
                 </geometry>
             </visual>
@@ -138,5 +187,7 @@
                 <origin rpy="0 0 0" xyz="0.0 0.0 -0.5475" />
                 <geometry>
-                    <mesh filename="package://lbr_description/meshes/iiwa7/collision/link_3.stl" />
+                    <mesh
+                        filename="package://lbr_description/meshes/iiwa7/collision/link_3.stl"
+                    />
                 </geometry>
             </collision>
@@ -151,10 +202,12 @@
                 lower="${joint_limits['A4']['lower'] * PI / 180}"
                 upper="${joint_limits['A4']['upper'] * PI / 180}"
-                velocity="${joint_limits['A4']['velocity'] * PI / 180}" />
+                velocity="${joint_limits['A4']['velocity'] * PI / 180}"
+            />
             <safety_controller
                 soft_lower_limit="${joint_limits['A4']['lower'] * PI / 180}"
                 soft_upper_limit="${joint_limits['A4']['upper'] * PI / 180}"
                 k_position="${joint_limits['A4']['velocity'] / joint_limits['A4']['safety_position_margin']}"
-                k_velocity="${joint_limits['A4']['k_velocity']}" />
+                k_velocity="${joint_limits['A4']['k_velocity']}"
+            />
             <dynamics damping="${joint_damping}" friction="${joint_friction}" />
         </joint>
@@ -163,11 +216,19 @@
                 <origin rpy="0 0 0" xyz="0.0 -0.039793 0.086944" />
                 <mass value="4.031989" />
-                <inertia ixx="0.031695" ixy="0.0" ixz="0.0" iyy="0.030079" iyz="-0.005889"
-                    izz="0.009665" />
+                <inertia
+                    ixx="0.031695"
+                    ixy="0.0"
+                    ixz="0.0"
+                    iyy="0.030079"
+                    iyz="-0.005889"
+                    izz="0.009665"
+                />
             </inertial>
             <visual>
                 <origin rpy="0 0 0" xyz="0.0 -0.0105 -0.74" />
                 <geometry>
-                    <mesh filename="package://lbr_description/meshes/iiwa7/visual/link_4.dae" />
+                    <mesh
+                        filename="package://lbr_description/meshes/iiwa7/visual/link_4.dae"
+                    />
                 </geometry>
             </visual>
@@ -175,5 +236,7 @@
                 <origin rpy="0 0 0" xyz="0.0 -0.0105 -0.74" />
                 <geometry>
-                    <mesh filename="package://lbr_description/meshes/iiwa7/collision/link_4.stl" />
+                    <mesh
+                        filename="package://lbr_description/meshes/iiwa7/collision/link_4.stl"
+                    />
                 </geometry>
             </collision>
@@ -188,10 +251,12 @@
                 lower="${joint_limits['A5']['lower'] * PI / 180}"
                 upper="${joint_limits['A5']['upper'] * PI / 180}"
-                velocity="${joint_limits['A5']['velocity'] * PI / 180}" />
+                velocity="${joint_limits['A5']['velocity'] * PI / 180}"
+            />
             <safety_controller
                 soft_lower_limit="${joint_limits['A5']['lower'] * PI / 180}"
                 soft_upper_limit="${joint_limits['A5']['upper'] * PI / 180}"
                 k_position="${joint_limits['A5']['velocity'] / joint_limits['A5']['safety_position_margin']}"
-                k_velocity="${joint_limits['A5']['k_velocity']}" />
+                k_velocity="${joint_limits['A5']['k_velocity']}"
+            />
             <dynamics damping="${joint_damping}" friction="${joint_friction}" />
         </joint>
@@ -200,11 +265,19 @@
                 <origin rpy="0 0 0" xyz="0.0 -0.029824 0.076267" />
                 <mass value="1.529239" />
-                <inertia ixx="0.008485" ixy="0.0" ixz="0.0" iyy="0.007136" iyz="0.002806"
-                    izz="0.003848" />
+                <inertia
+                    ixx="0.008485"
+                    ixy="0.0"
+                    ixz="0.0"
+                    iyy="0.007136"
+                    iyz="0.002806"
+                    izz="0.003848"
+                />
             </inertial>
             <visual>
                 <origin rpy="0 0 0" xyz="0.0 0.0 -0.9475" />
                 <geometry>
-                    <mesh filename="package://lbr_description/meshes/iiwa7/visual/link_5.dae" />
+                    <mesh
+                        filename="package://lbr_description/meshes/iiwa7/visual/link_5.dae"
+                    />
                 </geometry>
             </visual>
@@ -212,5 +285,7 @@
                 <origin rpy="0 0 0" xyz="0.0 0.0 -0.9475" />
                 <geometry>
-                    <mesh filename="package://lbr_description/meshes/iiwa7/collision/link_5.stl" />
+                    <mesh
+                        filename="package://lbr_description/meshes/iiwa7/collision/link_5.stl"
+                    />
                 </geometry>
             </collision>
@@ -225,10 +300,12 @@
                 lower="${joint_limits['A6']['lower'] * PI / 180}"
                 upper="${joint_limits['A6']['upper'] * PI / 180}"
-                velocity="${joint_limits['A6']['velocity'] * PI / 180}" />
+                velocity="${joint_limits['A6']['velocity'] * PI / 180}"
+            />
             <safety_controller
                 soft_lower_limit="${joint_limits['A6']['lower'] * PI / 180}"
                 soft_upper_limit="${joint_limits['A6']['upper'] * PI / 180}"
                 k_position="${joint_limits['A6']['velocity'] / joint_limits['A6']['safety_position_margin']}"
-                k_velocity="${joint_limits['A6']['k_velocity']}" />
+                k_velocity="${joint_limits['A6']['k_velocity']}"
+            />
             <dynamics damping="${joint_damping}" friction="${joint_friction}" />
         </joint>
@@ -237,11 +314,19 @@
                 <origin rpy="0 0 0" xyz="0.0 0.07102 0.00495" />
                 <mass value="2.403626" />
-                <inertia ixx="0.007067" ixy="0.0" ixz="0.0" iyy="0.006804" iyz="0.000311"
-                    izz="0.004629" />
+                <inertia
+                    ixx="0.007067"
+                    ixy="0.0"
+                    ixz="0.0"
+                    iyy="0.006804"
+                    iyz="0.000311"
+                    izz="0.004629"
+                />
             </inertial>
             <visual>
                 <origin rpy="0 0 0" xyz="0.0 0.0707 -1.14" />
                 <geometry>
-                    <mesh filename="package://lbr_description/meshes/iiwa7/visual/link_6.dae" />
+                    <mesh
+                        filename="package://lbr_description/meshes/iiwa7/visual/link_6.dae"
+                    />
                 </geometry>
             </visual>
@@ -249,5 +334,7 @@
                 <origin rpy="0 0 0" xyz="0.0 0.0707 -1.14" />
                 <geometry>
-                    <mesh filename="package://lbr_description/meshes/iiwa7/collision/link_6.stl" />
+                    <mesh
+                        filename="package://lbr_description/meshes/iiwa7/collision/link_6.stl"
+                    />
                 </geometry>
             </collision>
@@ -262,10 +349,12 @@
                 lower="${joint_limits['A7']['lower'] * PI / 180}"
                 upper="${joint_limits['A7']['upper'] * PI / 180}"
-                velocity="${joint_limits['A7']['velocity'] * PI / 180}" />
+                velocity="${joint_limits['A7']['velocity'] * PI / 180}"
+            />
             <safety_controller
                 soft_lower_limit="${joint_limits['A7']['lower'] * PI / 180}"
                 soft_upper_limit="${joint_limits['A7']['upper'] * PI / 180}"
                 k_position="${joint_limits['A7']['velocity'] / joint_limits['A7']['safety_position_margin']}"
-                k_velocity="${joint_limits['A7']['k_velocity']}" />
+                k_velocity="${joint_limits['A7']['k_velocity']}"
+            />
             <dynamics damping="${joint_damping}" friction="${joint_friction}" />
         </joint>
@@ -274,10 +363,19 @@
                 <origin rpy="0 0 0" xyz="3.0000e-06 -2.0000e-06 1.3782e-02" />
                 <mass value="0.259474" />
-                <inertia ixx="0.000171" ixy="0.0" ixz="0.0" iyy="0.000171" iyz="0.0" izz="0.000299" />
+                <inertia
+                    ixx="0.000171"
+                    ixy="0.0"
+                    ixz="0.0"
+                    iyy="0.000171"
+                    iyz="0.0"
+                    izz="0.000299"
+                />
             </inertial>
             <visual>
                 <origin rpy="0 0 0" xyz="0.0 0.0 -1.231" />
                 <geometry>
-                    <mesh filename="package://lbr_description/meshes/iiwa7/visual/link_7.dae" />
+                    <mesh
+                        filename="package://lbr_description/meshes/iiwa7/visual/link_7.dae"
+                    />
                 </geometry>
             </visual>
@@ -285,9 +383,11 @@
                 <origin rpy="0 0 0" xyz="0.0 0.0 -1.231" />
                 <geometry>
-                    <mesh filename="package://lbr_description/meshes/iiwa7/collision/link_7.stl" />
-                </geometry>
-            </collision>
-        </link>
-        <joint name="${robot_name}_joint_ee" type="fixed">
+                    <mesh
+                        filename="package://lbr_description/meshes/iiwa7/collision/link_7.stl"
+                    />
+                </geometry>
+            </collision>
+        </link>
+        <!-- <joint name="${robot_name}_joint_ee" type="fixed">
             <parent link="${robot_name}_link_7" />
             <child link="${robot_name}_link_ee" />
@@ -295,5 +395,5 @@
         </joint>
         <link name="${robot_name}_link_ee">
-        </link>
+        </link> -->
     </xacro:macro>
 </robot>
