Commit message: feat: new simulation world environment assemblence

File: lbr_description/urdf/iiwa7/iiwa7.xacro (robot description, xacro)
@@ -2,4 +2,18 @@
 <!-- top level -->
 <robot name="iiwa7" xmlns:xacro="http://www.ros.org/wiki/xacro">
+    <!-- propiedades rectangulo realidad-->
+    <xacro:property name="base_length" value="1.20" />   <!-- largo  X -->
+    <xacro:property name="base_width"  value="0.80" />   <!-- ancho  Y -->
+    <xacro:property name="base_height" value="1.00" />   <!-- alto   Z -->
+    <xacro:property name="base_mass"   value="40.0" />   <!-- kg       -->
+    <xacro:property name="robot_offset_x" value="0.40" /> <!-- extremo en X: (length/2 - margen) -->
+    <xacro:property name="robot_offset_y" value="0.0" />
+    <xacro:property name="base_ixx" value="5.333" />
+    <xacro:property name="base_iyy" value="5.600" />
+    <xacro:property name="base_izz" value="5.467" />
+    <xacro:property name="screen_offset_x"    value="-0.40" />
+    <xacro:property name="screen_offset_y"    value="0.0" />
+    <xacro:property name="screen_box_height"  value="0.20"  />
+    <xacro:property name="screen_panel_z"     value="0.20" />
     <!-- include the iiwa macro and controller -->
     <xacro:include filename="$(find lbr_description)/urdf/iiwa7/iiwa7.urdf.xacro" />
@@ -21,9 +35,110 @@
     will tipple https://github.com/lbr-stack/lbr_fri_ros2_stack/issues/230 -->
     <link name="world" />
+    <!-- esto estaba antes de los cambios (dejalo por si acaso o algo twin)-->
     <!--joint
         between <robot_name>_world_link and robot_name_link_0-->
-    <joint name="$(arg robot_name)_world_joint" type="fixed">
+<!--     <joint name="$(arg robot_name)_world_joint" type="fixed">
         <parent link="world" />
         <child link="$(arg robot_name)_link_0" />
+    </joint> -->
+    <!-- world base rectangular -->
+    <joint name="$(arg robot_name)_world_base_joint" type="fixed">
+        <parent link="world" />
+        <child  link="$(arg robot_name)_base_link" />
+        <origin xyz="0 0 ${base_height / 2}" rpy="0 0 0" />
+    </joint>
+    <link name="$(arg robot_name)_base_link">
+        <inertial>
+            <origin xyz="0 0 0" rpy="0 0 0" />
+            <mass value="${base_mass}" />
+            <inertia ixx="${base_ixx}" ixy="0.0" ixz="0.0"
+                    iyy="${base_iyy}" iyz="0.0"
+                    izz="${base_izz}" />
+        </inertial>
+        <visual>
+            <origin xyz="0 0 0" rpy="0 0 0" />
+            <geometry>
+                <box size="${base_length} ${base_width} ${base_height}" />
+            </geometry>
+            <material name="base_material">
+               <color rgba="0.1 0.3 0.6 1.0" />
+            </material>
+        </visual>
+        <collision>
+            <origin xyz="0 0 0" rpy="0 0 0" />
+            <geometry>
+                <box size="${base_length} ${base_width} ${base_height}" />
+            </geometry>
+        </collision>
+    </link>
+    <!-- Pantalla en el extremo opuesto al robot -->
+    <link name="$(arg robot_name)_screen_link">
+        <inertial>
+            <origin xyz="0 0 0" rpy="0 0 0" />
+            <mass value="3.0" />
+            <inertia ixx="0.05" ixy="0.0" ixz="0.0"
+                    iyy="0.03" iyz="0.0"
+                    izz="0.07" />
+        </inertial>
+        <!-- Caja base/soporte -->
+        <visual>
+            <origin xyz="0 0 ${screen_box_height / 2}" rpy="0 0 0" />
+            <geometry>
+                <box size="0.4375 0.0625 ${screen_box_height}" />
+            </geometry>
+            <material name="screen_base_material">
+                <color rgba="0.7 0.7 0.7 1.0" />
+            </material>
+        </visual>
+        <collision>
+            <origin xyz="0 0 ${screen_box_height / 2}" rpy="0 0 0" />
+            <geometry>
+                <box size="0.4375 0.0625 ${screen_box_height}" />
+            </geometry>
+        </collision>
+    </link>
+    <!-- Panel de la pantalla -->
+    <link name="$(arg robot_name)_screen_panel_link">
+        <inertial>
+            <origin xyz="0 0 0" rpy="0 0 0" />
+            <mass value="1.5" />
+            <inertia ixx="0.02" ixy="0.0" ixz="0.0"
+                    iyy="0.02" iyz="0.0"
+                    izz="0.01" />
+        </inertial>
+        <!-- Panel -->
+        <visual>
+            <origin xyz="0 0 0" rpy="0 0 0" />
+            <geometry>
+                <box size="0.4125 0.025 0.3125" />
+            </geometry>
+            <material name="screen_panel_material">
+                <color rgba="0.05 0.05 0.05 1.0" />
+            </material>
+        </visual>
+        <collision>
+            <origin xyz="0 0 0" rpy="0 0 0" />
+            <geometry>
+                <box size="0.4125 0.025 0.3125" />
+            </geometry>
+        </collision>
+    </link>
+    <!-- joint de la base de la pantalla la cosa esa gris-->
+    <joint name="$(arg robot_name)_base_screen_joint" type="fixed">
+        <parent link="$(arg robot_name)_base_link" />
+        <child  link="$(arg robot_name)_screen_link" />
+        <origin xyz="${screen_offset_x} ${screen_offset_y} ${base_height / 2}" rpy="0 0 1.5708" />
+    </joint>
+    <!-- Joint soporte panel inclinado-->
+    <joint name="$(arg robot_name)_screen_panel_joint" type="fixed">
+        <parent link="$(arg robot_name)_screen_link" />
+        <child  link="$(arg robot_name)_screen_panel_link" />
+        <origin xyz="0 0.075 ${screen_box_height + screen_panel_z * 0.5}" rpy="0.35 0 0" />
+    </joint>
+    <!-- base rectangular enganchado a lbr_link_0 -->
+    <joint name="$(arg robot_name)_base_robot_joint" type="fixed">
+        <parent link="$(arg robot_name)_base_link" />
+        <child  link="$(arg robot_name)_link_0" />
+        <origin xyz="${robot_offset_x} ${robot_offset_y} ${base_height / 2}" rpy="0 0 0" />
     </joint>
     <!-- macros for gazebo / mock / hardware -->
