Commit message: fix: corrected the joints

File: lbr_description/urdf/iiwa7/iiwa7.xacro (robot description, xacro)
@@ -177,4 +177,22 @@
     </joint>
     -->
+    <xacro:macro name="preserve_fixed" params="joint_name">
+        <gazebo reference="${joint_name}">
+            <preserveFixedJoint>true</preserveFixedJoint>
+        </gazebo>
+    </xacro:macro>
+    <xacro:preserve_fixed joint_name="lbr_world_base_joint" />
+    <xacro:preserve_fixed joint_name="lbr_base_robot_joint" />
+    <xacro:preserve_fixed joint_name="lbr_link_7_brida_cam_base_joint" />
+    <xacro:preserve_fixed joint_name="lbr_link_7_brida_cam_tip_joint" />
+    <!-- brida_cam_tip_ft45_base_joint ya está preservada vía ft_gazebo_plugin -->
+    <xacro:preserve_fixed joint_name="brida_cam_tip_ft45_tip_joint" />
+    <xacro:preserve_fixed joint_name="ft45_tip_brida_ft_base_joint" />
+    <xacro:preserve_fixed joint_name="ft45_tip_brida_ft_tip_joint" />
+    <xacro:preserve_fixed joint_name="brida_ft_tip_tool_body_joint" />
+    <xacro:preserve_fixed joint_name="brida_ft_tip_tool_body_tip_joint" />
+    <xacro:preserve_fixed joint_name="tool_sponge_joint" />
+    <xacro:preserve_fixed joint_name="tool_body_tip_tool_tip_joint" />
+    <xacro:preserve_fixed joint_name="lbr_joint_ee" />
     <!-- ============================================================ -->
     <!-- GAZEBO CONTACT/Collision SURFACES for links missing references -->

Commit message: rollback

File: lbr_description/urdf/iiwa7/iiwa7.xacro (robot description, xacro)
@@ -177,5 +177,5 @@
     </joint>
     -->
-    <xacro:macro name="preserve_fixed" params="joint_name">
+    <!-- <xacro:macro name="preserve_fixed" params="joint_name">
         <gazebo reference="${joint_name}">
             <preserveFixedJoint>true</preserveFixedJoint>
@@ -187,7 +187,6 @@
     <xacro:preserve_fixed joint_name="ft45_tip_brida_ft_base_joint" />
     <xacro:preserve_fixed joint_name="brida_ft_tip_tool_body_joint" />
-    <xacro:preserve_fixed joint_name="brida_ft_tip_tool_body_tip_joint" />
     <xacro:preserve_fixed joint_name="tool_sponge_joint" />
-    <xacro:preserve_fixed joint_name="lbr_joint_ee" />
+    <xacro:preserve_fixed joint_name="lbr_joint_ee" /> -->
     <!-- ============================================================ -->
     <!-- GAZEBO CONTACT/Collision SURFACES for links missing references -->

Commit message: fix(iiwa7): reactivar preserveFixedJoint + forzar self-collision DART
- Se reactiva la macro preserve_fixed y sus llamadas para todas las
  juntas fijas cuyo hijo termina en _base (world_base, base_robot,
  link_7_brida_cam_base, brida_cam_tip_ft45_base,
  ft45_tip_brida_ft_base, brida_ft_tip_tool_body, tool_sponge).
- Se añade brida_cam_tip_ft45_base_joint que faltaba en la lista
  original.
- Se elimina lbr_joint_ee por ser una junta _tip sin geometría de
  colisión.
- Se añade <dart><collision_detector>ode</collision_detector></dart>
  en el bloque <gazebo> del modelo para evitar que DART se salte
  self-collision entre pares ancestro/descendiente.

Sin preserveFixedJoint, el conversor URDF->SDF de Gazebo Ignition
fusiona todos los links conectados por juntas fijas en un solo cuerpo
rígido, haciendo que DART ignore las colisiones entre la cadena de
herramienta y el carrito/pantalla. Esto impedía que el test de
histéresis detectara fuerzas de contacto en el sensor FT.

File: lbr_description/urdf/iiwa7/iiwa7.xacro (robot description, xacro)
@@ -6,7 +6,11 @@
     <!-- between links welded via fixed joints within the same model.  -->
     <!-- false = self-collision ENABLED (links CAN collide).           -->
+    <!-- DART collision_detector=ode avoids ancestor/descendant skip.  -->
     <!-- ============================================================ -->
     <gazebo>
         <selfCollide>false</selfCollide>
+        <dart>
+            <collision_detector>ode</collision_detector>
+        </dart>
     </gazebo>
     <!-- caja, pasar a primitiva para la colision? ahorra computo creo-->
@@ -177,16 +181,28 @@
     </joint>
     -->
-    <!-- <xacro:macro name="preserve_fixed" params="joint_name">
+    <!-- ============================================================ -->
+    <!-- preserveFixedJoint: prevents Gazebo Ignition from merging     -->
+    <!-- links connected by fixed joints into a single rigid body.     -->
+    <!-- This is CRITICAL for collision detection between the tool     -->
+    <!-- chain (_base links) and the cart/screen.                      -->
+    <!-- Only _base joints are preserved (tip joints are empty dummies -->
+    <!-- that can be safely merged).                                   -->
+    <!-- ============================================================ -->
+    <xacro:macro name="preserve_fixed" params="joint_name">
         <gazebo reference="${joint_name}">
             <preserveFixedJoint>true</preserveFixedJoint>
         </gazebo>
     </xacro:macro>
+    <!-- Base structure: world ↔ base_link ↔ link_0 -->
     <xacro:preserve_fixed joint_name="lbr_world_base_joint" />
     <xacro:preserve_fixed joint_name="lbr_base_robot_joint" />
+    <!-- Tool chain: preserve all _base joints (child link ends in _base) -->
     <xacro:preserve_fixed joint_name="lbr_link_7_brida_cam_base_joint" />
+    <xacro:preserve_fixed joint_name="brida_cam_tip_ft45_base_joint" />
     <xacro:preserve_fixed joint_name="ft45_tip_brida_ft_base_joint" />
     <xacro:preserve_fixed joint_name="brida_ft_tip_tool_body_joint" />
     <xacro:preserve_fixed joint_name="tool_sponge_joint" />
-    <xacro:preserve_fixed joint_name="lbr_joint_ee" /> -->
+    <!-- Tip joints (child link ends in _tip) are NOT preserved: they  -->
+    <!-- carry no collision geometry and can be merged safely.          -->
     <!-- ============================================================ -->
     <!-- GAZEBO CONTACT/Collision SURFACES for links missing references -->
