Commit message: rollback

File: lbr_description/urdf/iiwa7/iiwa7.xacro (robot description, xacro)
@@ -1,17 +1,4 @@
 <?xml version="1.0" ?>
 <robot name="iiwa7" xmlns:xacro="http://www.ros.org/wiki/xacro">
-    <!-- ============================================================ -->
-    <!-- Explicitly enable self-collision for the entire model.        -->
-    <!-- Without this, Gazebo Ignition/DART may skip collision checks  -->
-    <!-- between links welded via fixed joints within the same model.  -->
-    <!-- false = self-collision ENABLED (links CAN collide).           -->
-    <!--                                                               -->
-    <!-- NOTE: the robot is now embedded in the world SDF at launch    -->
-    <!-- time (gazebo.launch.py) to work around gz-sim bug #3261 /     -->
-    <!-- #2957 where self_collide is ignored on runtime-spawned URDF.  -->
-    <!-- ============================================================ -->
-    <gazebo>
-        <selfCollide>false</selfCollide>
-    </gazebo>
     <!-- caja, pasar a primitiva para la colision? ahorra computo creo-->
     <xacro:property name="base_mass" value="40.0" />
@@ -181,33 +168,7 @@
     </joint>
     -->
-    <!-- ============================================================ -->
-    <!-- preserveFixedJoint: prevents Gazebo Ignition from merging     -->
-    <!-- links connected by fixed joints into a single rigid body.     -->
-    <!-- This is CRITICAL for collision detection between the tool     -->
-    <!-- chain (_base links) and the cart/screen.                      -->
-    <!-- Only _base joints are preserved (tip joints are empty dummies -->
-    <!-- that can be safely merged).                                   -->
-    <!-- ============================================================ -->
-    <xacro:macro name="preserve_fixed" params="joint_name">
-        <gazebo reference="${joint_name}">
-            <preserveFixedJoint>true</preserveFixedJoint>
-        </gazebo>
-    </xacro:macro>
     <!-- Base structure: world ↔ base_link ↔ link_0 -->
     <xacro:preserve_fixed joint_name="lbr_world_base_joint" />
     <xacro:preserve_fixed joint_name="lbr_base_robot_joint" />
-    <!-- Tool chain: preserve all _base joints (child link ends in _base) -->
-    <xacro:preserve_fixed joint_name="lbr_link_7_brida_cam_base_joint" />
-    <xacro:preserve_fixed joint_name="brida_cam_tip_ft45_base_joint" />
-    <xacro:preserve_fixed joint_name="ft45_tip_brida_ft_base_joint" />
-    <xacro:preserve_fixed joint_name="brida_ft_tip_tool_body_joint" />
-    <xacro:preserve_fixed joint_name="tool_sponge_joint" />
-    <!-- Tip joints (child link ends in _tip) are NOT preserved: they  -->
-    <!-- carry no collision geometry and can be merged safely.          -->
-    <!-- ============================================================ -->
-    <!-- GAZEBO CONTACT/Collision SURFACES for links missing references -->
-    <!-- Without these, Gazebo Ignition will not resolve contacts     -->
-    <!-- between the tool chain and the cart/screen.                   -->
-    <!-- ============================================================ -->
     <!-- Carrito / pantalla: superficie rígida (metal/plástico) -->
     <gazebo reference="$(arg robot_name)_base_link">

Commit message: feat: add independent screen_ghost SDF model for collision detection
The screen collision box in lbr_base_link was part of the same top-level
robot model, so the physics engine (ODE/Bullet in gz-sim) would skip
self-collision between the sponge tool and the screen — both belong to
the same <robot> tree. This meant no contact forces were generated for
the FT sensor's provideFeedback.

Instead of enabling self_collide (which risks ghost contacts between
adjacent arm links), we spawn a separate static SDF model at the same
world pose as the screen. As an independent rigid body, it collides
normally with the sponge tool.

Changes:
- New lbr_description/models/screen_ghost/model.sdf: static box with
  the same collision geometry (0.389x0.705x0.323) and contact params
  (kp=100k, kd=100, mu1=0.5, mu2=0.3) as the original screen.
- New lbr_description/models/screen_ghost/model.config for gz model DB.
- iiwa7.xacro: commented out the screen collision inside lbr_base_link
  to avoid double contact forces. The visual mesh is preserved.
- gazebo.launch.py: spawn screen_ghost via ros_gz_sim create with
  absolute world pose (-0.2195, 0, 0.8215), computed as
  screen_local_offset + base_link_to_world_offset.
  No namespace — it is a standalone world model, not part of the robot.

File: lbr_description/urdf/iiwa7/iiwa7.xacro (robot description, xacro)
@@ -105,11 +105,11 @@
             </geometry>
         </collision> -->
-        <!-- colisión extra para la pantalla (rectángulo) -->
-        <collision>
+        <!-- colisión de pantalla movida al modelo independiente screen_ghost -->
+        <!-- <collision>
             <origin xyz="-0.2195 0 0.1615" rpy="0 0 0" />
             <geometry>
                 <box size="0.389 0.705 0.323" />
             </geometry>
-        </collision>
+        </collision> -->
     </link>
     <joint name="$(arg robot_name)_base_robot_joint" type="fixed">

Commit message: chore: remove dead code from iiwa7.xacro
- Removed undefined <xacro:preserve_fixed> calls that referenced
  hardcoded 'lbr' prefix instead of the robot_name arg.
- Removed commented-out TCP dummy link/joint block.
- Removed <gazebo reference="base_link"> contact parameters: the
  link no longer has collision geometry (screen moved to screen_ghost
  model, big box already commented out).

File: lbr_description/urdf/iiwa7/iiwa7.xacro (robot description, xacro)
@@ -158,27 +158,4 @@
     <link name="$(arg robot_name)_link_ee">
     </link>
-    <!-- TCP alternativo fijo desde link_7 para IK -->
-    <!-- no uso el dummy para que no haya una duplicidad de los puntos TCP, sin cambios, no funciona la optimizacion igualmente -->
-    <!--
-    <link name="tool_tip_dummy" />
-    <joint name="$(arg robot_name)_link_7-tool_tip_dummy" type="fixed">
-        <parent link="tool_tip" />
-        <child link="tool_tip_dummy" />
-        <origin xyz="0 0 0" rpy="0 0 ${pi}" />
-    </joint>
-    -->
-    <!-- Base structure: world ↔ base_link ↔ link_0 -->
-    <xacro:preserve_fixed joint_name="lbr_world_base_joint" />
-    <xacro:preserve_fixed joint_name="lbr_base_robot_joint" />
-    <!-- Carrito / pantalla: superficie rígida (metal/plástico) -->
-    <gazebo reference="$(arg robot_name)_base_link">
-        <kp>100000.0</kp>          <!-- contact stiffness (N/m), alto = rígido -->
-        <kd>100.0</kd>             <!-- contact damping (N·s/m) -->
-        <mu1>0.5</mu1>             <!-- fricción estática -->
-        <mu2>0.3</mu2>             <!-- fricción dinámica -->
-        <maxVel>0.01</maxVel>      <!-- velocidad máxima de contacto -->
-        <minDepth>0.001</minDepth> <!-- penetración mínima antes de resolver -->
-        <maxContacts>4</maxContacts>
-    </gazebo>
     <!-- Brida cámara (extremo link_7) -->
     <gazebo reference="brida_cam_base">
