Commit message: fix: udpated colision for tooltip and sponges

File: lbr_description/models/tool/tool.xacro (robot description, xacro)
@@ -100,5 +100,5 @@
           <!--- forma primitiva para optimizar CPU, calculos propios -->
           <!-- TODO: revisar las dimensiones del cilindro para que se ajusten a la realidad -->
-            <cylinder radius="0.075" length="0.10" />
+            <cylinder radius="0.04" length="0.04" />
             <!-- <mesh filename="package://lbr_description/models/tool/meshes/collision/tool_base.stl"/> -->
           </geometry>
@@ -135,5 +135,5 @@
           <!--- forma primitiva para optimizar CPU, calculos propios -->
           <!-- TODO: revisar las dimensiones del cilindro para que se ajusten a la realidad -->
-            <cylinder radius="0.075" length="0.0524" />
+            <cylinder radius="0.04" length="0.04" />
             <!-- <mesh filename="package://lbr_description/models/tool/meshes/collision/tool_sponge_red.stl"/> -->
           </geometry>

Commit message: fix: updated length on sponge

File: lbr_description/models/tool/tool.xacro (robot description, xacro)
@@ -96,9 +96,9 @@
         </visual>
         <collision>
-          <origin xyz="0 0 0" rpy="0 0 0" />
+          <origin xyz="0 0 0" rpy="0 0 0.01" />
           <geometry>
           <!--- forma primitiva para optimizar CPU, calculos propios -->
           <!-- TODO: revisar las dimensiones del cilindro para que se ajusten a la realidad -->
-            <cylinder radius="0.04" length="0.04" />
+            <cylinder radius="0.04" length="0.02" />
             <!-- <mesh filename="package://lbr_description/models/tool/meshes/collision/tool_base.stl"/> -->
           </geometry>

Commit message: fix: updated length on sponge for collision detection

File: lbr_description/models/tool/tool.xacro (robot description, xacro)
@@ -96,5 +96,5 @@
         </visual>
         <collision>
-          <origin xyz="0 0 0" rpy="0 0 0.01" />
+          <origin xyz="0 0 0" rpy="0 0 -0.01" />
           <geometry>
           <!--- forma primitiva para optimizar CPU, calculos propios -->

Commit message: fix: updated sponge red for tooltip

File: lbr_description/models/tool/tool.xacro (robot description, xacro)
@@ -96,9 +96,9 @@
         </visual>
         <collision>
-          <origin xyz="0 0 0" rpy="0 0 -0.01" />
+          <origin xyz="0 0 0" rpy="0 0 0" />
           <geometry>
           <!--- forma primitiva para optimizar CPU, calculos propios -->
           <!-- TODO: revisar las dimensiones del cilindro para que se ajusten a la realidad -->
-            <cylinder radius="0.04" length="0.02" />
+            <cylinder radius="0.04" length="0.04" />
             <!-- <mesh filename="package://lbr_description/models/tool/meshes/collision/tool_base.stl"/> -->
           </geometry>
@@ -131,9 +131,9 @@
         </visual>
         <collision>
-          <origin xyz="0 0 0" rpy="0 0 0" />
+          <origin xyz="0 0 0" rpy="0 0 0.01" />
           <geometry>
           <!--- forma primitiva para optimizar CPU, calculos propios -->
           <!-- TODO: revisar las dimensiones del cilindro para que se ajusten a la realidad -->
-            <cylinder radius="0.04" length="0.04" />
+            <cylinder radius="0.04" length="0.02" />
             <!-- <mesh filename="package://lbr_description/models/tool/meshes/collision/tool_sponge_red.stl"/> -->
           </geometry>

Commit message: fix: new update on fixed joint for links

File: lbr_description/models/tool/tool.xacro (robot description, xacro)
@@ -96,5 +96,5 @@
         </visual>
         <collision>
-          <origin xyz="0 0 0" rpy="0 0 0" />
+          <origin xyz="0 0 0" rpy="0 0 -0.02" />
           <geometry>
           <!--- forma primitiva para optimizar CPU, calculos propios -->
@@ -131,5 +131,5 @@
         </visual>
         <collision>
-          <origin xyz="0 0 0" rpy="0 0 0.01" />
+          <origin xyz="0 0 0" rpy="0 0 -0.01" />
           <geometry>
           <!--- forma primitiva para optimizar CPU, calculos propios -->

Commit message: update: update joints

File: lbr_description/models/tool/tool.xacro (robot description, xacro)
@@ -96,5 +96,5 @@
         </visual>
         <collision>
-          <origin xyz="0 0 0" rpy="0 0 -0.02" />
+          <origin xyz="0 0 0" rpy="0 0 -0.04" />
           <geometry>
           <!--- forma primitiva para optimizar CPU, calculos propios -->
@@ -131,5 +131,5 @@
         </visual>
         <collision>
-          <origin xyz="0 0 0" rpy="0 0 -0.01" />
+          <origin xyz="0 0 0" rpy="0 0 -0.02" />
           <geometry>
           <!--- forma primitiva para optimizar CPU, calculos propios -->

Commit message: test

File: lbr_description/models/tool/tool.xacro (robot description, xacro)
@@ -131,5 +131,5 @@
         </visual>
         <collision>
-          <origin xyz="0 0 0" rpy="0 0 -0.02" />
+          <origin xyz="0 0 0" rpy="0 0 -0.10" />
           <geometry>
           <!--- forma primitiva para optimizar CPU, calculos propios -->

Commit message: fix: updated collision on xyz positions

File: lbr_description/models/tool/tool.xacro (robot description, xacro)
@@ -96,9 +96,9 @@
         </visual>
         <collision>
-          <origin xyz="0 0 0" rpy="0 0 -0.04" />
+          <origin xyz="0 0 -0.03" rpy="0 0 0" />
           <geometry>
           <!--- forma primitiva para optimizar CPU, calculos propios -->
           <!-- TODO: revisar las dimensiones del cilindro para que se ajusten a la realidad -->
-            <cylinder radius="0.04" length="0.04" />
+            <cylinder radius="0.03" length="0.03" />
             <!-- <mesh filename="package://lbr_description/models/tool/meshes/collision/tool_base.stl"/> -->
           </geometry>
@@ -131,9 +131,9 @@
         </visual>
         <collision>
-          <origin xyz="0 0 0" rpy="0 0 -0.10" />
+          <origin xyz="0 0 -0.1" rpy="0 0 0" />
           <geometry>
           <!--- forma primitiva para optimizar CPU, calculos propios -->
           <!-- TODO: revisar las dimensiones del cilindro para que se ajusten a la realidad -->
-            <cylinder radius="0.04" length="0.02" />
+            <cylinder radius="0.045" length="0.02" />
             <!-- <mesh filename="package://lbr_description/models/tool/meshes/collision/tool_sponge_red.stl"/> -->
           </geometry>

Commit message: update cylinder collision

File: lbr_description/models/tool/tool.xacro (robot description, xacro)
@@ -96,5 +96,5 @@
         </visual>
         <collision>
-          <origin xyz="0 0 -0.03" rpy="0 0 0" />
+          <origin xyz="0 0 0.03" rpy="0 0 0" />
           <geometry>
           <!--- forma primitiva para optimizar CPU, calculos propios -->
@@ -131,5 +131,5 @@
         </visual>
         <collision>
-          <origin xyz="0 0 -0.1" rpy="0 0 0" />
+          <origin xyz="0 0 0.01" rpy="0 0 0" />
           <geometry>
           <!--- forma primitiva para optimizar CPU, calculos propios -->

Commit message: updated: radius for tcp tools

File: lbr_description/models/tool/tool.xacro (robot description, xacro)
@@ -96,5 +96,5 @@
         </visual>
         <collision>
-          <origin xyz="0 0 0.03" rpy="0 0 0" />
+          <origin xyz="0 0 0.015" rpy="0 0 0" />
           <geometry>
           <!--- forma primitiva para optimizar CPU, calculos propios -->
@@ -131,5 +131,5 @@
         </visual>
         <collision>
-          <origin xyz="0 0 0.01" rpy="0 0 0" />
+          <origin xyz="0 0 0.015" rpy="0 0 0" />
           <geometry>
           <!--- forma primitiva para optimizar CPU, calculos propios -->
