Commit message: fix: sponge effort for limits new

File: lbr_description/models/tool/tool.xacro (robot description, xacro)
@@ -173,12 +173,23 @@
       </link>
       <link name="${name}_tip"/>
-      <joint name="${parent}_${name}_tip_joint" type="fixed">
+      <!-- <joint name="${parent}_${name}_tip_joint" type="fixed">
         <origin xyz="0 0 0.036" rpy="0 0 0"/>
         <parent link="${name}_base"/>
         <child link="${name}_tip"/>
-      </joint>
+      </joint> -->
+      <joint name="${robot_name}_tip_joint" type="revolute">
+       <origin xyz="0 0 0.036" rpy="0 0 0"/>
+       <parent link="${name}_base"/>
+       <child link="${name}_tip"/>
+       <axis xyz="0.0 0.0 1.0" />
+        <limit
+                effort="1000000"
+                lower="0"
+                upper="0"
+                velocity="0" />
+    </joint>
     </xacro:macro>
     <xacro:macro name="conditioning_sponge_red" params="name parent *origin">
-      <joint name="${name}_sponge_joint" type="fixed">
+      <joint name="${name}_sponge_joint" type="revolute">
         <xacro:insert_block name="origin" />
         <parent link="${parent}"/>
@@ -205,8 +216,19 @@
       </link>
     <link name="${name}_tip"/>
-    <joint name="${parent}_${name}_tip_joint" type="fixed">
+    <!-- <joint name="${parent}_${name}_tip_joint" type="fixed">
       <origin xyz="0 0 0.0262" rpy="0 0 0"/>
       <parent link="${name}_base"/>
       <child link="${name}_tip"/>
+    </joint -->
+    <joint name="${robot_name}_tip_joint" type="revolute">
+      <origin xyz="0 0 0.0262" rpy="0 0 0"/>
+      <parent link="${name}_base"/>
+      <child link="${name}_tip"/>
+      <axis xyz="0.0 0.0 1.0" />
+        <limit
+                effort="1000000"
+                lower="0"
+                upper="0"
+                velocity="0" />
     </joint>
     </xacro:macro>

File: lbr_description/urdf/iiwa14/iiwa14.xacro (robot description, xacro)
@@ -160,30 +160,30 @@
     </link>
     <!-- Brida cámara (extremo link_7) -->
-    <gazebo reference="brida_cam_base">
+    <!-- <gazebo reference="brida_cam_base">
         <kp>100000.0</kp>
         <kd>100.0</kd>
         <mu1>0.5</mu1>
         <mu2>0.3</mu2>
-    </gazebo>
+    </gazebo> -->
     <!-- Sensor FT45 -->
-    <gazebo reference="ft45_base">
+    <!-- <gazebo reference="ft45_base">
         <kp>100000.0</kp>
         <kd>100.0</kd>
         <mu1>0.5</mu1>
         <mu2>0.3</mu2>
-    </gazebo>
+    </gazebo> -->
     <!-- Brida FT -->
-    <gazebo reference="brida_ft_base">
+    <!-- <gazebo reference="brida_ft_base">
         <kp>100000.0</kp>
         <kd>100.0</kd>
         <mu1>0.5</mu1>
         <mu2>0.3</mu2>
-    </gazebo>
+    </gazebo> -->
     <!-- Tool body (base de la esponja) -->
     <gazebo reference="tool_body_base">
-        <kp>10000.0</kp>
-        <kd>100.0</kd>
-        <mu1>0.5</mu1>
-        <mu2>0.3</mu2>
+        <kp>5000.0</kp>
+        <kd>50.0</kd>
+        <mu1>1.0</mu1>
+        <mu2>0.8</mu2>
     </gazebo>
     <!-- Esponja (tool): material blando, kp/kd más bajos para simular deformabilidad -->

Commit message: fix: enhance repair_sponge_red macro with multi-layer dynamics and adjust properties

File: lbr_description/models/tool/tool.xacro (robot description, xacro)
@@ -113,7 +113,9 @@
     </xacro:macro>
     <xacro:macro name="repair_sponge_red" params="name parent *origin
-                 spring_stiffness:=2000.0
-                 spring_damping:=5.0
-                 max_compression:=0.006">
+                 layer_radius:=0.045
+                 layer_length:=0.00333
+                 layer1_stiffness:=4000.0 layer1_damping:=6.0 layer1_max_compression:=0.001
+                 layer2_stiffness:=2500.0 layer2_damping:=4.0 layer2_max_compression:=0.0015
+                 layer3_stiffness:=1200.0 layer3_damping:=3.0 layer3_max_compression:=0.002">
       <!-- Montaje rigido de la base de la esponja al tool_body -->
       <joint name="${name}_mount_joint" type="fixed">
@@ -135,5 +137,5 @@
         </visual>
         <!-- Nucleo rigido: coleccion mas pequena/anidada que la esponja real.
-             El "colchon" de compresion lo aporta el link movil de abajo -->
+             El "colchon" de compresion lo aportan las 3 capas de abajo -->
         <collision>
           <origin xyz="0 0 0.0075" rpy="0 0 0" />
@@ -143,32 +145,103 @@
         </collision>
       </link>
-      <!-- Joint prismatico con resorte articulado: esto simula el material blando.
-           DART no soporta compliance de contacto real vía kp/kd, pero sí soporta
-           spring_stiffness/spring_reference en joints vía axis/dynamics. -->
-      <joint name="${name}_sponge_prismatic_joint" type="prismatic">
-        <origin xyz="0 0 0.0075" rpy="0 0 0" />
+      <!-- ==========================================================
+           CAPAS DE LA ESPONJA (discretizacion en serie).
+           Cada capa es su propio link con su propio joint prismatico +
+           resorte (dynamics spring_stiffness/spring_reference). Las 3
+           capas se apilan de forma CONSECUTIVA (cada joint desplaza
+           exactamente "layer_length" desde el tope de la capa anterior),
+           por lo que las colisiones NUNCA se solapan entre si.
+           Capa 1 = mas cercana al nucleo rigido (mas rigida, simula la
+                    base comprimida de la esponja).
+           Capa 3 = capa de contacto con la superficie (mas blanda, es
+                    la que primero se deforma al tocar).
+           NOTA: si en pruebas ves que spring_stiffness/spring_reference
+           no producen fuerza real en gz-sim (bug conocido, ver
+           https://github.com/gazebosim/gz-sim/issues/2520), la
+           alternativa es sustituir estos 3 joints por un system plugin
+           tipo SpringSystem que aplique la fuerza explicitamente sobre
+           cada joint en cada paso de simulacion.
+           ========================================================== -->
+      <!-- Capa 1: pegada al nucleo rigido -->
+      <joint name="${name}_layer1_joint" type="prismatic">
+        <origin xyz="0 0 0.0115" rpy="0 0 0" />
         <parent link="${name}_base"/>
-        <child link="${name}_base2"/>
+        <child link="${name}_layer1"/>
         <axis xyz="0 0 1" />
-        <limit lower="-${max_compression}" upper="0" effort="50" velocity="0.5" />
-        <dynamics damping="${spring_damping}" spring_stiffness="${spring_stiffness}" spring_reference="0.0" />
-      </joint>
-      <link name="${name}_base2">
-        <inertial>
-          <mass value="0.02" />
-          <origin xyz="0 0 0.005" rpy="0 0 0" />
-          <inertia ixx="0.0002" ixy="0.0" ixz="0.0" iyy="0.0002" iyz="0.0" izz="0.0002" />
-        </inertial>
-        <visual>
-          <origin xyz="0 0 0.0075" rpy="0 0 0" />
-          <geometry>
-            <cylinder radius="0.045" length="0.01" />
-          </geometry>
-        </visual>
-        <!-- Coleccion "real" de la esponja: la que toca la pantalla y se comprime -->
-        <collision>
-          <origin xyz="0 0 0.0075" rpy="0 0 0" />
-          <geometry>
-            <cylinder radius="0.045" length="0.01" />
+        <limit lower="-${layer1_max_compression}" upper="0" effort="50" velocity="0.5" />
+        <dynamics damping="${layer1_damping}" spring_stiffness="${layer1_stiffness}" spring_reference="0.0" />
+      </joint>
+      <link name="${name}_layer1">
+        <inertial>
+          <mass value="0.007" />
+          <origin xyz="0 0 ${layer_length/2}" rpy="0 0 0" />
+          <inertia ixx="7e-05" ixy="0.0" ixz="0.0" iyy="7e-05" iyz="0.0" izz="7e-05" />
+        </inertial>
+        <visual>
+          <origin xyz="0 0 ${layer_length/2}" rpy="0 0 0" />
+          <geometry>
+            <cylinder radius="${layer_radius}" length="${layer_length}" />
+          </geometry>
+        </visual>
+        <collision>
+          <origin xyz="0 0 ${layer_length/2}" rpy="0 0 0" />
+          <geometry>
+            <cylinder radius="${layer_radius}" length="${layer_length}" />
+          </geometry>
+        </collision>
+      </link>
+      <!-- Capa 2: intermedia -->
+      <joint name="${name}_layer2_joint" type="prismatic">
+        <origin xyz="0 0 ${layer_length}" rpy="0 0 0" />
+        <parent link="${name}_layer1"/>
+        <child link="${name}_layer2"/>
+        <axis xyz="0 0 1" />
+        <limit lower="-${layer2_max_compression}" upper="0" effort="50" velocity="0.5" />
+        <dynamics damping="${layer2_damping}" spring_stiffness="${layer2_stiffness}" spring_reference="0.0" />
+      </joint>
+      <link name="${name}_layer2">
+        <inertial>
+          <mass value="0.007" />
+          <origin xyz="0 0 ${layer_length/2}" rpy="0 0 0" />
+          <inertia ixx="7e-05" ixy="0.0" ixz="0.0" iyy="7e-05" iyz="0.0" izz="7e-05" />
+        </inertial>
+        <visual>
+          <origin xyz="0 0 ${layer_length/2}" rpy="0 0 0" />
+          <geometry>
+            <cylinder radius="${layer_radius}" length="${layer_length}" />
+          </geometry>
+        </visual>
+        <collision>
+          <origin xyz="0 0 ${layer_length/2}" rpy="0 0 0" />
+          <geometry>
+            <cylinder radius="${layer_radius}" length="${layer_length}" />
+          </geometry>
+        </collision>
+      </link>
+      <!-- Capa 3: capa de contacto (la que toca la superficie) -->
+      <joint name="${name}_layer3_joint" type="prismatic">
+        <origin xyz="0 0 ${layer_length}" rpy="0 0 0" />
+        <parent link="${name}_layer2"/>
+        <child link="${name}_layer3"/>
+        <axis xyz="0 0 1" />
+        <limit lower="-${layer3_max_compression}" upper="0" effort="50" velocity="0.5" />
+        <dynamics damping="${layer3_damping}" spring_stiffness="${layer3_stiffness}" spring_reference="0.0" />
+      </joint>
+      <link name="${name}_layer3">
+        <inertial>
+          <mass value="0.007" />
+          <origin xyz="0 0 ${layer_length/2}" rpy="0 0 0" />
+          <inertia ixx="7e-05" ixy="0.0" ixz="0.0" iyy="7e-05" iyz="0.0" izz="7e-05" />
+        </inertial>
+        <visual>
+          <origin xyz="0 0 ${layer_length/2}" rpy="0 0 0" />
+          <geometry>
+            <cylinder radius="${layer_radius}" length="${layer_length}" />
+          </geometry>
+        </visual>
+        <collision>
+          <origin xyz="0 0 ${layer_length/2}" rpy="0 0 0" />
+          <geometry>
+            <cylinder radius="${layer_radius}" length="${layer_length}" />
           </geometry>
         </collision>
@@ -176,6 +249,6 @@
     <link name="${name}_tip"/>
     <joint name="${parent}_${name}_tip_joint" type="fixed">
-      <origin xyz="0 0 0.0162" rpy="0 0 0"/>
-      <parent link="${name}_base2"/>
+      <origin xyz="0 0 ${layer_length}" rpy="0 0 0"/>
+      <parent link="${name}_layer3"/>
       <child link="${name}_tip"/>
     </joint>

Commit message: fix: remove unused joint and link definitions in repair_sponge_red macro for cleaner code

File: lbr_description/models/tool/tool.xacro (robot description, xacro)
@@ -52,28 +52,4 @@
         </collision>
       </link>
-      <!-- <joint name="${name}_base_joint" type="fixed">
-        <origin xyz="0 0 0.056" rpy="0 0 0"/>
-        <parent link="${name}_brida"/>
-        <child link="${name}_base"/>
-      </joint>
-      <link name="${name}_base">
-        <inertial>
-          <mass value="1.1" />
-          <origin xyz="-0.011278 -0.001814 0.052275" rpy="0 0 0" />
-          <inertia ixx="0.001483" ixy="-0.000145" ixz="-0.000314" iyy="0.002166" iyz="-9.2e-05" izz="0.001375" />
-        </inertial>
-        <visual>
-          <origin xyz="0 0 0" rpy="0 0 0"/>
-          <geometry>
-                  <mesh filename="package://kuka_control/models/tool/meshes/visual/Airos350CV_red_sponge.dae"/>
-          </geometry>
-        </visual>
-        <collision>
-          <origin xyz="0 0 0" rpy="0 0 0" />
-          <geometry>
-            <mesh filename="package://kuka_control/models/tool/meshes/collision/Airos350CV_red_sponge.stl"/>
-          </geometry>
-        </collision>
-      </link> -->
     </xacro:macro>
     <xacro:macro name="repair_tool_iiwa" params="name parent *origin">
@@ -98,8 +74,5 @@
           <origin xyz="0 0 0.015" rpy="0 0 0" />
           <geometry>
-          <!--- forma primitiva para optimizar CPU, calculos propios -->
-          <!-- TODO: revisar las dimensiones del cilindro para que se ajusten a la realidad -->
             <cylinder radius="0.03" length="0.03" />
-            <!-- <mesh filename="package://lbr_description/models/tool/meshes/collision/tool_base.stl"/> -->
           </geometry>
         </collision>
@@ -114,17 +87,16 @@
     <xacro:macro name="repair_sponge_red" params="name parent *origin
                  layer_radius:=0.045
-                 layer_length:=0.00333
+                 layer_length:=0.006667
                  layer1_stiffness:=4000.0 layer1_damping:=6.0 layer1_max_compression:=0.001
                  layer2_stiffness:=2500.0 layer2_damping:=4.0 layer2_max_compression:=0.0015
                  layer3_stiffness:=1200.0 layer3_damping:=3.0 layer3_max_compression:=0.002">
-      <!-- Montaje rigido de la base de la esponja al tool_body -->
-      <joint name="${name}_mount_joint" type="fixed">
-        <xacro:insert_block name="origin" />
-        <parent link="${parent}"/>
-        <child link="${name}_base"/>
-      </joint>
-      <link name="${name}_base">
-        <inertial>
-          <mass value="0.055" />
+      <joint name="${name}_sponge_joint" type="fixed">
+        <xacro:insert_block name="origin" />
+        <parent link="${parent}"/>
+        <child link="${name}_base"/>
+      </joint>
+      <link name="${name}_base">
+        <inertial>
+          <mass value="0.110" />
           <origin xyz="-0.009159 -0.01474 0.093085" rpy="0 0 0" />
           <inertia ixx="0.002444" ixy="-0.000123" ixz="-0.000103" iyy="0.003024" iyz="-5.1e-05" izz="0.001237" />
@@ -136,34 +108,7 @@
           </geometry>
         </visual>
-        <!-- Nucleo rigido: coleccion mas pequena/anidada que la esponja real.
-             El "colchon" de compresion lo aportan las 3 capas de abajo -->
-        <collision>
-          <origin xyz="0 0 0.0075" rpy="0 0 0" />
-          <geometry>
-            <cylinder radius="0.040" length="0.008" />
-          </geometry>
-        </collision>
-      </link>
-      <!-- ==========================================================
-           CAPAS DE LA ESPONJA (discretizacion en serie).
-           Cada capa es su propio link con su propio joint prismatico +
-           resorte (dynamics spring_stiffness/spring_reference). Las 3
-           capas se apilan de forma CONSECUTIVA (cada joint desplaza
-           exactamente "layer_length" desde el tope de la capa anterior),
-           por lo que las colisiones NUNCA se solapan entre si.
-           Capa 1 = mas cercana al nucleo rigido (mas rigida, simula la
-                    base comprimida de la esponja).
-           Capa 3 = capa de contacto con la superficie (mas blanda, es
-                    la que primero se deforma al tocar).
-           NOTA: si en pruebas ves que spring_stiffness/spring_reference
-           no producen fuerza real en gz-sim (bug conocido, ver
-           https://github.com/gazebosim/gz-sim/issues/2520), la
-           alternativa es sustituir estos 3 joints por un system plugin
-           tipo SpringSystem que aplique la fuerza explicitamente sobre
-           cada joint en cada paso de simulacion.
-           ========================================================== -->
-      <!-- Capa 1: pegada al nucleo rigido -->
+      </link>
       <joint name="${name}_layer1_joint" type="prismatic">
-        <origin xyz="0 0 0.0115" rpy="0 0 0" />
+        <origin xyz="0 0 0.005" rpy="0 0 0" />
         <parent link="${name}_base"/>
         <child link="${name}_layer1"/>
@@ -174,22 +119,15 @@
       <link name="${name}_layer1">
         <inertial>
-          <mass value="0.007" />
+          <mass value="0.0075" />
           <origin xyz="0 0 ${layer_length/2}" rpy="0 0 0" />
           <inertia ixx="7e-05" ixy="0.0" ixz="0.0" iyy="7e-05" iyz="0.0" izz="7e-05" />
         </inertial>
-        <visual>
+        <collision>
           <origin xyz="0 0 ${layer_length/2}" rpy="0 0 0" />
           <geometry>
             <cylinder radius="${layer_radius}" length="${layer_length}" />
           </geometry>
-        </visual>
-        <collision>
-          <origin xyz="0 0 ${layer_length/2}" rpy="0 0 0" />
-          <geometry>
-            <cylinder radius="${layer_radius}" length="${layer_length}" />
-          </geometry>
-        </collision>
-      </link>
-      <!-- Capa 2: intermedia -->
+        </collision>
+      </link>
       <joint name="${name}_layer2_joint" type="prismatic">
         <origin xyz="0 0 ${layer_length}" rpy="0 0 0" />
@@ -202,22 +140,15 @@
       <link name="${name}_layer2">
         <inertial>
-          <mass value="0.007" />
+          <mass value="0.0075" />
           <origin xyz="0 0 ${layer_length/2}" rpy="0 0 0" />
           <inertia ixx="7e-05" ixy="0.0" ixz="0.0" iyy="7e-05" iyz="0.0" izz="7e-05" />
         </inertial>
-        <visual>
+        <collision>
           <origin xyz="0 0 ${layer_length/2}" rpy="0 0 0" />
           <geometry>
             <cylinder radius="${layer_radius}" length="${layer_length}" />
           </geometry>
-        </visual>
-        <collision>
-          <origin xyz="0 0 ${layer_length/2}" rpy="0 0 0" />
-          <geometry>
-            <cylinder radius="${layer_radius}" length="${layer_length}" />
-          </geometry>
-        </collision>
-      </link>
-      <!-- Capa 3: capa de contacto (la que toca la superficie) -->
+        </collision>
+      </link>
       <joint name="${name}_layer3_joint" type="prismatic">
         <origin xyz="0 0 ${layer_length}" rpy="0 0 0" />
@@ -230,14 +161,8 @@
       <link name="${name}_layer3">
         <inertial>
-          <mass value="0.007" />
+          <mass value="0.0075" />
           <origin xyz="0 0 ${layer_length/2}" rpy="0 0 0" />
           <inertia ixx="7e-05" ixy="0.0" ixz="0.0" iyy="7e-05" iyz="0.0" izz="7e-05" />
         </inertial>
-        <visual>
-          <origin xyz="0 0 ${layer_length/2}" rpy="0 0 0" />
-          <geometry>
-            <cylinder radius="${layer_radius}" length="${layer_length}" />
-          </geometry>
-        </visual>
         <collision>
           <origin xyz="0 0 ${layer_length/2}" rpy="0 0 0" />
@@ -249,5 +174,5 @@
     <link name="${name}_tip"/>
     <joint name="${parent}_${name}_tip_joint" type="fixed">
-      <origin xyz="0 0 ${layer_length}" rpy="0 0 0"/>
+      <origin xyz="0 0 0.007867" rpy="0 0 0"/>
       <parent link="${name}_layer3"/>
       <child link="${name}_tip"/>
@@ -280,9 +205,4 @@
       </link>
       <link name="${name}_tip"/>
-      <!-- <joint name="${parent}_${name}_tip_joint" type="fixed">
-        <origin xyz="0 0 0.036" rpy="0 0 0"/>
-        <parent link="${name}_base"/>
-        <child link="${name}_tip"/>
-      </joint> -->
       <joint name="${robot_name}_tip_joint" type="revolute">
        <origin xyz="0 0 0.036" rpy="0 0 0"/>
@@ -323,9 +243,4 @@
       </link>
     <link name="${name}_tip"/>
-    <!-- <joint name="${parent}_${name}_tip_joint" type="fixed">
-      <origin xyz="0 0 0.0262" rpy="0 0 0"/>
-      <parent link="${name}_base"/>
-      <child link="${name}_tip"/>
-    </joint -->
     <joint name="${robot_name}_tip_joint" type="revolute">
       <origin xyz="0 0 0.0262" rpy="0 0 0"/>
