Commit message: fix: enhance repair_sponge_red macro with spring dynamics and adjust mass properties

File: lbr_description/models/tool/tool_backup.xacro (robot description, xacro)
@@ -112,17 +112,13 @@
       </joint>
     </xacro:macro>
-    <xacro:macro name="repair_sponge_red" params="name parent *origin
-                 spring_stiffness:=2000.0
-                 spring_damping:=5.0
-                 max_compression:=0.006">
-      <!-- Montaje rigido de la base de la esponja al tool_body -->
-      <joint name="${name}_mount_joint" type="fixed">
-        <xacro:insert_block name="origin" />
-        <parent link="${parent}"/>
-        <child link="${name}_base"/>
-      </joint>
-      <link name="${name}_base">
-        <inertial>
-          <mass value="0.055" />
+    <xacro:macro name="repair_sponge_red" params="name parent *origin">
+      <joint name="${name}_sponge_joint" type="fixed">
+        <xacro:insert_block name="origin" />
+        <parent link="${parent}"/>
+        <child link="${name}_base"/>
+      </joint>
+      <link name="${name}_base">
+        <inertial>
+          <mass value="0.110" />
           <origin xyz="-0.009159 -0.01474 0.093085" rpy="0 0 0" />
           <inertia ixx="0.002444" ixy="-0.000123" ixz="-0.000103" iyy="0.003024" iyz="-5.1e-05" izz="0.001237" />
@@ -134,41 +130,11 @@
           </geometry>
         </visual>
-        <!-- Nucleo rigido: coleccion mas pequena/anidada que la esponja real.
-             El "colchon" de compresion lo aporta el link movil de abajo -->
-        <collision>
-          <origin xyz="0 0 0.0075" rpy="0 0 0" />
-          <geometry>
-            <cylinder radius="0.040" length="0.008" />
-          </geometry>
-        </collision>
-      </link>
-      <!-- Joint prismatico con resorte articulado: esto simula el material blando.
-           DART no soporta compliance de contacto real vía kp/kd, pero sí soporta
-           spring_stiffness/spring_reference en joints vía axis/dynamics. -->
-      <joint name="${name}_sponge_prismatic_joint" type="prismatic">
-        <origin xyz="0 0 0.0075" rpy="0 0 0" />
-        <parent link="${name}_base"/>
-        <child link="${name}_base2"/>
-        <axis xyz="0 0 1" />
-        <limit lower="-${max_compression}" upper="0" effort="50" velocity="0.5" />
-        <dynamics damping="${spring_damping}" spring_stiffness="${spring_stiffness}" spring_reference="0.0" />
-      </joint>
-      <link name="${name}_base2">
-        <inertial>
-          <mass value="0.02" />
-          <origin xyz="0 0 0.005" rpy="0 0 0" />
-          <inertia ixx="0.0002" ixy="0.0" ixz="0.0" iyy="0.0002" iyz="0.0" izz="0.0002" />
-        </inertial>
-        <visual>
-          <origin xyz="0 0 0.0075" rpy="0 0 0" />
-          <geometry>
-            <cylinder radius="0.045" length="0.01" />
-          </geometry>
-        </visual>
-        <!-- Coleccion "real" de la esponja: la que toca la pantalla y se comprime -->
-        <collision>
-          <origin xyz="0 0 0.0075" rpy="0 0 0" />
-          <geometry>
-            <cylinder radius="0.045" length="0.01" />
+        <collision>
+          <origin xyz="0 0 0.015" rpy="0 0 0" />
+          <geometry>
+          <!--- forma primitiva para optimizar CPU, calculos propios -->
+          <!-- TODO: revisar las dimensiones del cilindro para que se ajusten a la realidad -->
+            <cylinder radius="0.045" length="0.02" />
+            <!-- <mesh filename="package://lbr_description/models/tool/meshes/collision/tool_sponge_red.stl"/> -->
           </geometry>
         </collision>
@@ -176,6 +142,6 @@
     <link name="${name}_tip"/>
     <joint name="${parent}_${name}_tip_joint" type="fixed">
-      <origin xyz="0 0 0.0162" rpy="0 0 0"/>
-      <parent link="${name}_base2"/>
+      <origin xyz="0 0 0.0262" rpy="0 0 0"/>
+      <parent link="${name}_base"/>
       <child link="${name}_tip"/>
     </joint>
