Commit message: fix: commented link_ee

File: lbr_description/urdf/iiwa14/iiwa14.urdf.xacro (robot description, xacro)
@@ -289,5 +289,5 @@
             </collision>
         </link>
-        <joint name="${robot_name}_joint_ee" type="fixed">
+        <!-- <joint name="${robot_name}_joint_ee" type="fixed">
             <parent link="${robot_name}_link_7" />
             <child link="${robot_name}_link_ee" />
@@ -295,5 +295,5 @@
         </joint>
         <link name="${robot_name}_link_ee">
-        </link>
+        </link> -->
     </xacro:macro>
 </robot>
