Commit message: fix: iiwa14 support

File: lbr_description/urdf/iiwa14/iiwa14.xacro (robot description, xacro)
@@ -1,9 +1,20 @@
-<?xml version="1.0"?>
+<?xml version="1.0" ?>
 <!-- top level -->
 <robot name="iiwa14" xmlns:xacro="http://www.ros.org/wiki/xacro">
+    <!-- caja, pasar a primitiva para la colision? ahorra computo creo-->
+    <xacro:property name="base_mass" value="40.0" />
+    <xacro:property name="robot_offset_x" value="0.40" />
+    <xacro:property name="robot_offset_y" value="0.0" />
+    <xacro:property name="base_ixx" value="5.333" />
+    <xacro:property name="base_iyy" value="5.600" />
+    <xacro:property name="base_izz" value="5.467" />
     <!-- include the iiwa macro and controller -->
     <xacro:include filename="$(find lbr_description)/urdf/iiwa14/iiwa14.urdf.xacro" />
     <xacro:include filename="$(find lbr_description)/gazebo/lbr_gazebo.xacro" />
     <xacro:include filename="$(find lbr_description)/ros2_control/lbr_system_interface.xacro" />
+    <xacro:include
+        filename="$(find lbr_description)/models/ft_sensor/real_ft_sensor_macro.xacro"
+    />
+    <xacro:include filename="$(find lbr_description)/models/tool/tool.xacro" />
     <!-- arguments -->
     <xacro:arg name="robot_name" default="lbr" />
@@ -18,12 +29,93 @@
         name="initial_joint_positions_path"
         default="$(find lbr_description)/ros2_control/initial_joint_positions.yaml" />
+    <xacro:macro
+        name="ft_gazebo_plugin"
+        params="ft_joint_name topic_name update_rate:='1000' noise_stddev_force:='0.01' noise_stddev_torque:='0.001'"
+    >
+        <gazebo reference="${ft_joint_name}">
+            <preserveFixedJoint>true</preserveFixedJoint>
+            <sensor name="ft_sensor" type="force_torque">
+                <always_on>true</always_on>
+                <update_rate>${update_rate}</update_rate>
+                <visualize>false</visualize>
+                <force_torque>
+                    <frame>child</frame>
+                    <measure_direction>child_to_parent</measure_direction>
+                    <force>
+                        <x><noise type="gaussian"><mean>0.0</mean><stddev
+                                >${noise_stddev_force}</stddev></noise></x>
+                        <y><noise type="gaussian"><mean>0.0</mean><stddev
+                                >${noise_stddev_force}</stddev></noise></y>
+                        <z><noise type="gaussian"><mean>0.0</mean><stddev
+                                >${noise_stddev_force}</stddev></noise></z>
+                    </force>
+                    <torque>
+                        <x><noise type="gaussian"><mean>0.0</mean><stddev
+                                >${noise_stddev_torque}</stddev></noise></x>
+                        <y><noise type="gaussian"><mean>0.0</mean><stddev
+                                >${noise_stddev_torque}</stddev></noise></y>
+                        <z><noise type="gaussian"><mean>0.0</mean><stddev
+                                >${noise_stddev_torque}</stddev></noise></z>
+                    </torque>
+                </force_torque>
+                <topic>${topic_name}</topic>
+                <plugin
+                    filename="gz-sim-forcetorque-system"
+                    name="gz::sim::systems::ForceTorque"
+                />
+            </sensor>
+        </gazebo>
+    </xacro:macro>
     <!-- KDL requires a link without inertia / Gazebo requires a connection to world link or robot
     will tipple https://github.com/lbr-stack/lbr_fri_ros2_stack/issues/230 -->
     <link name="world" />
-    <!--joint
-        between <robot_name>_world_link and robot_name_link_0-->
+    <!-- base_link (carrito) entre world y link_0 -->
+    <link name="$(arg robot_name)_base_link">
+        <inertial>
+            <origin xyz="0 0 0" rpy="0 0 0" />
+            <mass value="${base_mass}" />
+            <inertia
+                ixx="${base_ixx}"
+                ixy="0.0"
+                ixz="0.0"
+                iyy="${base_iyy}"
+                iyz="0.0"
+                izz="${base_izz}"
+            />
+        </inertial>
+        <visual>
+            <origin xyz="0 0 0" rpy="0 0 0" />
+            <geometry>
+                <mesh
+                    filename="package://lbr_description/meshes/iiwa14/carrito_azul/Cuerpo_carro_1.dae"
+                />
+            </geometry>
+        </visual>
+        <!-- caja simplificada para tratar de optimizar el codigo -->
+        <!-- <collision>
+            <origin xyz="0 0 -0.33" rpy="0 0 0" />
+            <geometry>
+                <box size="1.055 0.705 0.660" />
+            </geometry>
+        </collision> -->
+        <!-- colisión de pantalla movida al modelo independiente screen_ghost -->
+        <!-- <collision>
+            <origin xyz="-0.2195 0 0.1615" rpy="0 0 0" />
+            <geometry>
+                <box size="0.389 0.705 0.323" />
+            </geometry>
+        </collision> -->
+    </link>
+    <!-- joint between world and base_link -->
     <joint name="$(arg robot_name)_world_joint" type="fixed">
         <parent link="world" />
+        <child link="$(arg robot_name)_base_link" />
+        <origin xyz="0 0 0.660" rpy="0 0 0" />
+    </joint>
+    <!-- joint between base_link and link_0 -->
+    <joint name="$(arg robot_name)_base_robot_joint" type="fixed">
+        <parent link="$(arg robot_name)_base_link" />
         <child link="$(arg robot_name)_link_0" />
+        <origin xyz="${robot_offset_x} ${robot_offset_y} 0" rpy="0 0 ${pi/2}" />
     </joint>
     <!-- macros for gazebo / mock / hardware -->
@@ -38,3 +130,71 @@
         robot_name="$(arg robot_name)"
         joint_limits_path="$(arg joint_limits_path)" />
+    <!-- cadena: link_7 → brida_cam → ft45 → brida_ft → tool_body → sponge = TCP -->
+    <xacro:brida_cam parent="$(arg robot_name)_link_7" name="brida_cam">
+        <origin xyz="0 0 0.035" rpy="0 0 0" />
+    </xacro:brida_cam>
+    <xacro:ft45 parent="brida_cam_tip" name="ft45">
+        <origin xyz="0 0 0" rpy="0 0 ${pi}" />
+    </xacro:ft45>
+    <!-- plugin FT sobre joint: brida_cam_tip_ft45_base_joint -->
+    <xacro:ft_gazebo_plugin
+        ft_joint_name="brida_cam_tip_ft45_base_joint"
+        topic_name="ft_sensor/wrench"
+        update_rate="200"
+    /> <!-- bajado la frecuencia de actualizacion para optimizar, sin cambios -->
+    <xacro:brida_ft parent="ft45_tip" name="brida_ft">
+        <origin xyz="0 0 0" rpy="0 0 0" />
+    </xacro:brida_ft>
+    <xacro:repair_tool_iiwa name="tool_body" parent="brida_ft_tip">
+        <origin xyz="0 0 0" rpy="0 0 0" />
+    </xacro:repair_tool_iiwa>
+    <xacro:repair_sponge_red name="tool" parent="tool_body_tip">
+        <origin xyz="0 0 0" rpy="0 0 ${pi}" />
+    </xacro:repair_sponge_red>
+    <joint name="$(arg robot_name)_joint_ee" type="fixed">
+        <parent link="tool_tip" />
+        <child link="$(arg robot_name)_link_ee" />
+        <origin xyz="0 0 0" rpy="0 0 0" />
+    </joint>
+    <link name="$(arg robot_name)_link_ee">
+    </link>
+    <!-- Brida cámara (extremo link_7) -->
+    <gazebo reference="brida_cam_base">
+        <kp>100000.0</kp>
+        <kd>100.0</kd>
+        <mu1>0.5</mu1>
+        <mu2>0.3</mu2>
+    </gazebo>
+    <!-- Sensor FT45 -->
+    <gazebo reference="ft45_base">
+        <kp>100000.0</kp>
+        <kd>100.0</kd>
+        <mu1>0.5</mu1>
+        <mu2>0.3</mu2>
+    </gazebo>
+    <!-- Brida FT -->
+    <gazebo reference="brida_ft_base">
+        <kp>100000.0</kp>
+        <kd>100.0</kd>
+        <mu1>0.5</mu1>
+        <mu2>0.3</mu2>
+    </gazebo>
+    <!-- Tool body (base de la esponja) -->
+    <gazebo reference="tool_body_base">
+        <kp>100000.0</kp>
+        <kd>100.0</kd>
+        <mu1>0.5</mu1>
+        <mu2>0.3</mu2>
+    </gazebo>
+    <!-- Esponja (tool): material blando, kp/kd más bajos para simular deformabilidad -->
+    <gazebo reference="tool_base">
+        <provideFeedback>true</provideFeedback>
+        <kp>5000.0</kp>            <!-- stiffness bajo = esponja blanda -->
+        <kd>50.0</kd>              <!-- damping moderado -->
+        <mu1>1.0</mu1>             <!-- fricción alta esponja-pantalla -->
+        <mu2>0.8</mu2>
+        <maxVel>0.01</maxVel>
+        <minDepth>0.0001</minDepth>
+        <maxContacts>6</maxContacts>
+    </gazebo>
 </robot>

Commit message: docs: colisiones pantalla

File: lbr_description/urdf/iiwa14/iiwa14.xacro (robot description, xacro)
@@ -93,10 +93,10 @@
         </visual>
         <!-- caja simplificada para tratar de optimizar el codigo -->
-        <!-- <collision>
+        <collision>
             <origin xyz="0 0 -0.33" rpy="0 0 0" />
             <geometry>
                 <box size="1.055 0.705 0.660" />
             </geometry>
-        </collision> -->
+        </collision>
         <!-- colisión de pantalla movida al modelo independiente screen_ghost -->
         <!-- <collision>

Commit message: update 0.0.0 position to see datashet

File: lbr_description/urdf/iiwa14/iiwa14.xacro (robot description, xacro)
@@ -93,17 +93,17 @@
         </visual>
         <!-- caja simplificada para tratar de optimizar el codigo -->
-        <collision>
+        <!-- <collision>
             <origin xyz="0 0 -0.33" rpy="0 0 0" />
             <geometry>
                 <box size="1.055 0.705 0.660" />
             </geometry>
-        </collision>
+        </collision> -->
         <!-- colisión de pantalla movida al modelo independiente screen_ghost -->
-        <!-- <collision>
+        <collision>
             <origin xyz="-0.2195 0 0.1615" rpy="0 0 0" />
             <geometry>
                 <box size="0.389 0.705 0.323" />
             </geometry>
-        </collision> -->
+        </collision>
     </link>
     <!-- joint between world and base_link -->

Commit message: updated for demo_static.py

File: lbr_description/urdf/iiwa14/iiwa14.xacro (robot description, xacro)
@@ -2,18 +2,6 @@
 <!-- top level -->
 <robot name="iiwa14" xmlns:xacro="http://www.ros.org/wiki/xacro">
-    <!-- caja, pasar a primitiva para la colision? ahorra computo creo-->
-    <xacro:property name="base_mass" value="40.0" />
-    <xacro:property name="robot_offset_x" value="0.40" />
-    <xacro:property name="robot_offset_y" value="0.0" />
-    <xacro:property name="base_ixx" value="5.333" />
-    <xacro:property name="base_iyy" value="5.600" />
-    <xacro:property name="base_izz" value="5.467" />
     <!-- include the iiwa macro and controller -->
-    <xacro:include filename="$(find lbr_description)/urdf/iiwa14/iiwa14.urdf.xacro" />
-    <xacro:include filename="$(find lbr_description)/gazebo/lbr_gazebo.xacro" />
-    <xacro:include filename="$(find lbr_description)/ros2_control/lbr_system_interface.xacro" />
-    <xacro:include
-        filename="$(find lbr_description)/models/ft_sensor/real_ft_sensor_macro.xacro"
-    />
+    <xacro:include filename="$(find lbr_description)/models/ft_sensor/real_ft_sensor_macro.xacro" />
     <xacro:include filename="$(find lbr_description)/models/tool/tool.xacro" />
     <!-- arguments -->
@@ -70,123 +58,43 @@
     will tipple https://github.com/lbr-stack/lbr_fri_ros2_stack/issues/230 -->
     <link name="world" />
-    <!-- base_link (carrito) entre world y link_0 -->
-    <link name="$(arg robot_name)_base_link">
-        <inertial>
-            <origin xyz="0 0 0" rpy="0 0 0" />
-            <mass value="${base_mass}" />
-            <inertia
-                ixx="${base_ixx}"
-                ixy="0.0"
-                ixz="0.0"
-                iyy="${base_iyy}"
-                iyz="0.0"
-                izz="${base_izz}"
-            />
-        </inertial>
-        <visual>
-            <origin xyz="0 0 0" rpy="0 0 0" />
-            <geometry>
-                <mesh
-                    filename="package://lbr_description/meshes/iiwa14/carrito_azul/Cuerpo_carro_1.dae"
-                />
-            </geometry>
-        </visual>
-        <!-- caja simplificada para tratar de optimizar el codigo -->
-        <!-- <collision>
-            <origin xyz="0 0 -0.33" rpy="0 0 0" />
-            <geometry>
-                <box size="1.055 0.705 0.660" />
-            </geometry>
-        </collision> -->
-        <!-- colisión de pantalla movida al modelo independiente screen_ghost -->
-        <collision>
-            <origin xyz="-0.2195 0 0.1615" rpy="0 0 0" />
-            <geometry>
-                <box size="0.389 0.705 0.323" />
-            </geometry>
-        </collision>
-    </link>
-    <!-- joint between world and base_link -->
-    <joint name="$(arg robot_name)_world_joint" type="fixed">
-        <parent link="world" />
-        <child link="$(arg robot_name)_base_link" />
-        <origin xyz="0 0 0.660" rpy="0 0 0" />
-    </joint>
-    <!-- joint between base_link and link_0 -->
-    <joint name="$(arg robot_name)_base_robot_joint" type="fixed">
-        <parent link="$(arg robot_name)_base_link" />
-        <child link="$(arg robot_name)_link_0" />
-        <origin xyz="${robot_offset_x} ${robot_offset_y} 0" rpy="0 0 ${pi/2}" />
-    </joint>
-    <!-- macros for gazebo / mock / hardware -->
-    <xacro:lbr_gazebo robot_name="$(arg robot_name)" />
-    <xacro:lbr_system_interface
-        robot_name="$(arg robot_name)"
-        mode="$(arg mode)"
-        system_config_path="$(arg system_config_path)"
-        initial_joint_positions_path="$(arg initial_joint_positions_path)" />
     <!-- iiwa description -->
-    <xacro:iiwa14
-        robot_name="$(arg robot_name)"
-        joint_limits_path="$(arg joint_limits_path)" />
-    <!-- cadena: link_7 → brida_cam → ft45 → brida_ft → tool_body → sponge = TCP -->
-    <xacro:brida_cam parent="$(arg robot_name)_link_7" name="brida_cam">
-        <origin xyz="0 0 0.035" rpy="0 0 0" />
-    </xacro:brida_cam>
-    <xacro:ft45 parent="brida_cam_tip" name="ft45">
+    <xacro:ft45 parent="world" name="ft45">
         <origin xyz="0 0 0" rpy="0 0 ${pi}" />
     </xacro:ft45>
-    <!-- plugin FT sobre joint: brida_cam_tip_ft45_base_joint -->
+    <!-- plugin FT sobre joint: world_ft45_base_joint -->
     <xacro:ft_gazebo_plugin
-        ft_joint_name="brida_cam_tip_ft45_base_joint"
+        ft_joint_name="world_ft45_base_joint"
         topic_name="ft_sensor/wrench"
         update_rate="200"
     /> <!-- bajado la frecuencia de actualizacion para optimizar, sin cambios -->
-    <xacro:brida_ft parent="ft45_tip" name="brida_ft">
+      <joint name="sensor_sponge_joint" type="fixed">
         <origin xyz="0 0 0" rpy="0 0 0" />
-    </xacro:brida_ft>
-    <xacro:repair_tool_iiwa name="tool_body" parent="brida_ft_tip">
-        <origin xyz="0 0 0" rpy="0 0 0" />
-    </xacro:repair_tool_iiwa>
-    <xacro:repair_sponge_red name="tool" parent="tool_body_tip">
-        <origin xyz="0 0 0" rpy="0 0 ${pi}" />
-    </xacro:repair_sponge_red>
-    <joint name="$(arg robot_name)_joint_ee" type="fixed">
-        <parent link="tool_tip" />
-        <child link="$(arg robot_name)_link_ee" />
-        <origin xyz="0 0 0" rpy="0 0 0" />
-    </joint>
-    <link name="$(arg robot_name)_link_ee">
-    </link>
-    <!-- Brida cámara (extremo link_7) -->
-    <!-- <gazebo reference="brida_cam_base">
-        <kp>100000.0</kp>
-        <kd>100.0</kd>
-        <mu1>0.5</mu1>
-        <mu2>0.3</mu2>
-    </gazebo> -->
-    <!-- Sensor FT45 -->
-    <!-- <gazebo reference="ft45_base">
-        <kp>100000.0</kp>
-        <kd>100.0</kd>
-        <mu1>0.5</mu1>
-        <mu2>0.3</mu2>
-    </gazebo> -->
-    <!-- Brida FT -->
-    <!-- <gazebo reference="brida_ft_base">
-        <kp>100000.0</kp>
-        <kd>100.0</kd>
-        <mu1>0.5</mu1>
-        <mu2>0.3</mu2>
-    </gazebo> -->
-    <!-- Tool body (base de la esponja) -->
-    <gazebo reference="tool_body_base">
-        <kp>5000.0</kp>
-        <kd>50.0</kd>
-        <mu1>1.0</mu1>
-        <mu2>0.8</mu2>
-    </gazebo>
+        <parent link="ft45_tip"/>
+        <child link="sponge_base"/>
+      </joint>
+      <link name="sponge_base">
+        <inertial>
+          <mass value="0.110" />
+          <origin xyz="-0.009159 -0.01474 0.093085" rpy="0 0 0" />
+          <inertia ixx="0.002444" ixy="-0.000123" ixz="-0.000103" iyy="0.003024" iyz="-5.1e-05" izz="0.001237" />
+        </inertial>
+        <visual>
+          <origin xyz="0 0 0" rpy="0 0 0"/>
+          <geometry>
+            <mesh filename="package://lbr_description/models/tool/meshes/visual/tool_sponge_red.dae"/>
+          </geometry>
+        </visual>
+        <collision>
+          <origin xyz="0 0 0.015" rpy="0 0 0" />
+          <geometry>
+          <!--- forma primitiva para optimizar CPU, calculos propios -->
+          <!-- TODO: revisar las dimensiones del cilindro para que se ajusten a la realidad -->
+            <cylinder radius="0.045" length="0.02" />
+            <!-- <mesh filename="package://lbr_description/models/tool/meshes/collision/tool_sponge_red.stl"/> -->
+          </geometry>
+        </collision>
+      </link>
     <!-- Esponja (tool): material blando, kp/kd más bajos para simular deformabilidad -->
-    <gazebo reference="tool_base">
+    <gazebo reference="sponge_base">
         <provideFeedback>true</provideFeedback>
         <kp>5000.0</kp>            <!-- stiffness bajo = esponja blanda -->

Commit message: add ft45_base and ft45_tip links with corresponding joints in iiwa14.xacro

File: lbr_description/urdf/iiwa14/iiwa14.xacro (robot description, xacro)
@@ -58,14 +58,49 @@
     will tipple https://github.com/lbr-stack/lbr_fri_ros2_stack/issues/230 -->
     <link name="world" />
-    <!-- iiwa description -->
-    <xacro:ft45 parent="world" name="ft45">
+    <!-- sensor base fixed to world -->
+    <link name="ft45_base">
+        <inertial>
+            <mass value="0.15"/>
+            <origin xyz="0 0 0.0105" rpy="0 0 0"/>
+            <xacro:cylinder_inertia_def radius="0.0225" length="0.021" mass="0.15"/>
+        </inertial>
+        <visual>
+            <origin xyz="0 0 0" rpy="0 0 0"/>
+            <geometry>
+                <mesh filename="package://lbr_description/models/ft_sensor/meshes/visual/FT45.dae"/>
+            </geometry>
+        </visual>
+        <collision>
+            <origin xyz="0 0 0" rpy="0 0 0"/>
+            <geometry>
+                <cylinder radius="0.0225" length="0.021"/>
+            </geometry>
+        </collision>
+    </link>
+    <joint name="world_ft45_base_joint" type="fixed">
         <origin xyz="0 0 0" rpy="0 0 ${pi}" />
-    </xacro:ft45>
-    <!-- plugin FT sobre joint: world_ft45_tip_joint -->
+        <parent link="world"/>
+        <child link="ft45_base"/>
+    </joint>
+    <link name="ft45_tip">
+        <inertial>
+            <mass value="0.001"/>
+            <origin xyz="0 0 0" rpy="0 0 0"/>
+            <inertia ixx="1e-06" ixy="0" ixz="0" iyy="1e-06" iyz="0" izz="1e-06"/>
+        </inertial>
+    </link>
+    <!-- FT measurement joint: dynamic, locked -->
+    <joint name="ft45_sensor_joint" type="revolute">
+        <origin xyz="0 0 0.021" rpy="0 0 0"/>
+        <parent link="ft45_base"/>
+        <child link="ft45_tip"/>
+        <axis xyz="0 0 1"/>
+        <limit effort="1000" velocity="0" lower="0" upper="0"/>
+    </joint>
     <xacro:ft_gazebo_plugin
-        ft_joint_name="world_ft45_base_joint"
+        ft_joint_name="ft45_sensor_joint"
         topic_name="ft_sensor/wrench"
         update_rate="200"
-    /> <!-- bajado la frecuencia de actualizacion para optimizar, sin cambios -->
+    />
       <joint name="sensor_sponge_joint" type="fixed">
         <origin xyz="0 0 0" rpy="0 0 0" />
